File: nuled/pcb/nuled.kicad_sch (KiCad schematic)
At the start: 12 parts, among them J1 POWERSUPPLY, J3 USB C power supply, J4 LED strip out, SW1 Push-button

Commit message: schematics and documentation
Parts:
- removed J1: POWERSUPPLY, symbol Connector:Conn_01x02_Socket
- removed J5: ~, symbol nuled:ESP32C3-DevKit-Mini-1
- added C1, C12, C13, C16, C3, C6, C8: 0.1u, Capacitor_SMD:C_0201_0603Metric, symbol Device:C
- added C17, C18, C2: 22u, Capacitor_SMD:C_0201_0603Metric, symbol Device:C
- added C19: 470u/10V (20%), Capacitor_Tantalum_SMD:CP_EIA-3528-12_Kemet-T, symbol Device:C_Polarized
- added C20: 22u, Capacitor_Tantalum_SMD:CP_EIA-3528-12_Kemet-T, symbol Device:C
- added C21: 0.1u, Capacitor_Tantalum_SMD:CP_EIA-3528-12_Kemet-T, symbol Device:C
- added C22: 47u, Capacitor_SMD:C_0201_0603Metric, symbol Device:C
- added C23, C24: 47u/16V (X7R), Capacitor_SMD:C_0201_0603Metric, symbol Device:C
- added C4: 4.7u, Capacitor_SMD:C_0201_0603Metric, symbol Device:C
- added C5: 1u/16V (10%), Capacitor_SMD:C_0201_0603Metric, symbol Device:C
- added C7: 10u, Capacitor_SMD:C_0201_0603Metric, symbol Device:C
- added D1, D5: APT1608EC, Diode_SMD:D_0603_1608Metric, symbol Device:LED
- added D10, D11: BAV99, Package_TO_SOT_SMD:SOT-23, symbol Diode:BAV99
- added D2: APT1608YC, Diode_SMD:D_0603_1608Metric, symbol Device:LED
- added D3, D4: APT1608MGC, Diode_SMD:D_0603_1608Metric, symbol Device:LED
- added D8, D9: SMBJ5.0CA, Diode_SMD:D_SMA, symbol Diode:SMAJ5.0CA
- added J2: External supply, TerminalBlock_RND:TerminalBlock_RND_205-00232_1x02_P5.08mm_Horizontal, symbol Connector:Screw_Terminal_01x02
- added J3: Conn_01x09_Pin, symbol Connector:Conn_01x09_Pin
- added J5: Ext.switch, Connector_PinHeader_2.54mm:PinHeader_1x02_P2.54mm_Vertical, symbol Connector:Conn_01x02_Pin
- added J6: PJ-327A0-SMT, Connector_Audio:Jack_3.5mm_PJ320D_Horizontal, symbol Connector_Audio:AudioJack3
- added J7: LED strip 2, Connector_PinHeader_2.54mm:PinHeader_1x03_P2.54mm_Horizontal, symbol Connector:Screw_Terminal_01x03
- added J8: 5V 10A output, Connector_PinHeader_2.54mm:PinHeader_1x03_P2.54mm_Horizontal, symbol Connector:Screw_Terminal_01x02
- added Q1, Q2, Q3: DMP6180SK3-13, Package_TO_SOT_SMD:TO-252-2, symbol Simulation_SPICE:PMOS
- added Q4, Q5, Q6, Q7, Q8: SI2302, Package_TO_SOT_SMD:SOT-23, symbol Device:Q_NMOS_GDS
- added Q9: CJ2333, Package_TO_SOT_SMD:TO-252-2, symbol Simulation_SPICE:PMOS
- added R10, R11, R12, R15, R17, R19, R22, R28, R30, R31, R32, R34, R36, R37: 10k, Resistor_SMD:R_0201_0603Metric, symbol Device:R
- added R13, R14, R16, R18, R20, R33, R35: 1k, Resistor_SMD:R_0201_0603Metric, symbol Device:R
- added R21: 910k (1%), Resistor_SMD:R_0201_0603Metric, symbol Device:R
- added R23, R24: 1M, Resistor_SMD:R_0201_0603Metric, symbol Device:R
- added R25: 100k, Resistor_SMD:R_0201_0603Metric, symbol Device:R
- added R26: 47k, Resistor_SMD:R_0201_0603Metric, symbol Device:R
- added R27: 22k, Resistor_SMD:R_0201_0603Metric, symbol Device:R
- added R38: 220, Resistor_SMD:R_0201_0603Metric, symbol Device:R
- added R4: 100, Resistor_SMD:R_0201_0603Metric, symbol Device:R
- added R6, R7: 22 (1%), Resistor_SMD:R_0201_0603Metric, symbol Device:R
- added R8, R9: 0(1%), Resistor_SMD:R_0201_0603Metric, symbol Device:R
- added RV1: 3314J-1-103E, Potentiometer_SMD:Potentiometer_Bourns_3314J_Vertical, symbol Device:R_Potentiometer_Trim
- added TP1: EN/CHIP_PU, symbol Connector:TestPoint
- added TP2: GPIO0/USB_MODE_2, symbol Connector:TestPoint
- added TP3: GPIO1/USB_MODE_1, symbol Connector:TestPoint
- added TP4: U0TXD, symbol Connector:TestPoint
- added TP5: U0RXD, symbol Connector:TestPoint
- added TP6: GPIO7/~{VCONN_FAULT}, symbol Connector:TestPoint
- added TP7: GPIO9/BOOT, symbol Connector:TestPoint
- added U1: TPD2EUSB30, Package_TO_SOT_SMD:Texas_DRT-3, symbol Power_Protection:TPD2EUSB30
- added U2: AMS1117-3.3, Package_TO_SOT_SMD:SOT-223-3_TabPin2, symbol Regulator_Linear:AMS1117-3.3
- added U3: CP2102N-A02-GQFN28R, Package_DFN_QFN:QFN-28-1EP_5x5mm_P0.5mm_EP3.35x3.35mm, symbol Interface_USB:CP2102N-Axx-xQFN28
- added U4: ESP32-C3-MINI-1, PCM_Espressif:ESP32-C3-MINI-1, symbol PCM_Espressif:ESP32-C3-MINI-1
- added U5: TUSB321, Package_DFN_QFN:Texas_X2QFN-12_1.6x1.6mm_P0.4mm, symbol Interface_USB:TUSB321
- added U6: SN74LVC1T45DBVR, Package_SO:VSSOP-8_2.3x2mm_P0.5mm, symbol Logic_LevelTranslator:SN74LVC2T45DCUR
- C11: renamed from C1; value 1mF -> 470u/10V (20%); footprint (none) -> Capacitor_Tantalum_SMD:CP_EIA-3528-12_Kemet-T; Part (none) -> RVT1A471M0607
- C14: renamed from C2; value 0.1 -> 0.1u; footprint (none) -> Capacitor_SMD:C_0201_0603Metric; symbol Device:C_Polarized -> Device:C
- J1: renamed from J3; value USB C power supply -> U262-161N-4BVC11; footprint (none) -> Connector_USB:USB_C_Receptacle_XKB_U262-16XN-4BVC11
- J4: value LED strip out -> LED strip 1; footprint (none) -> Connector_PinHeader_2.54mm:PinHeader_1x03_P2.54mm_Horizontal
- R1: value R -> 100k; footprint (none) -> Resistor_SMD:R_0201_0603Metric
- R2: value 5k1 -> 100; footprint (none) -> Resistor_SMD:R_0201_0603Metric
- R29: renamed from R4; footprint (none) -> Resistor_SMD:R_0201_0603Metric
- R3: value 5k1 -> 100k; footprint (none) -> Resistor_SMD:R_0201_0603Metric
- R5: value R -> 1k; footprint (none) -> Resistor_SMD:R_0201_0603Metric
- SW1: value Push-button -> ???
Connections:
- net +5V: now also J4.3 (Pin_3), R2.2, R3.1, C1.1, C13.1, C17.2, C18.1, C18.2, C19.1, C20.1, C21.1, J7.1 (Pin_1), J8.1 (Pin_1), Q1.3 (S), Q3.1 (D), R13.1, R4.2, U2.3 (VI), U6.1 (VCCA); no longer J1.A4 (VBUS), J1.A9 (VBUS), J1.B4 (VBUS), J1.B9 (VBUS), J4.1 (Pin_1), R1.1
- net GND: now also J4.1 (Pin_1), R1.2, C1.2, C12.2, C13.2, C16.2, C19.2, C2.2, C20.2, C21.2, C22.2, C3.2, C4.2, C5.2, C6.2, C7.2, C8.2, D1.1 (K), D10.1 (K), D11.1 (K), D2.1 (K), D8.2 (A2), D9.2 (A2), J2.1 (Pin_1), J3.1 (Pin_1), J3.4 (Pin_4), J3.7 (Pin_7), J5.2 (Pin_2), J6.S, J7.3 (Pin_3), J8.2 (Pin_2), Q6.3 (S), Q7.3 (S), Q8.3 (S), R15.2, R17.2, R19.2, R22.2, R23.2, R24.2, R25.2, R26.1, R32.2, R34.2, R35.2, RV1.3, U1.3 (GND), U2.1 (GND), U3.29 (GND), U3.3 (GND), U4.1 (GND), U4.11 (GND), U4.14 (GND), U4.2 (GND), U4.36 (GND), U4.37 (GND), U4.38 (GND), U4.39 (GND), U4.40 (GND), U4.41 (GND), U4.42 (GND), U4.43 (GND), U4.44 (GND), U4.45 (GND), U4.46 (GND), U4.47 (GND), U4.48 (GND), U4.49 (GND), U4.50 (GND), U4.51 (GND), U4.52 (GND), U4.53 (GND), U5.10 (GND), U6.4 (GND), U6.5 (DIR); no longer J4.3 (Pin_3), R2.2
- net at R2.1: now also Q2.2 (G); no longer J1.A5 (CC1)
- net USB_UP: now reaches J1.A6 (D+)
- net USB_UP: now also J1.B6 (D+), R7.1, U1.1 (D+)
- net USB_DN: now reaches J1.A7 (D-)
- net USB_DN: now also J1.B7 (D-), R6.1, U1.2 (D-)
- net CC2: now reaches J1.B5 (CC2)
- net CC2: now also U5.2 (CC2); no longer R3.1
- net +3.3V: now reaches R5.1
- net +3.3V: now also C12.1, C2.1, C3.1, C4.1, C6.1, C7.1, D10.2 (A), D11.2 (A), J3.3 (Pin_3), J3.6 (Pin_6), J3.9 (Pin_9), R12.2, R14.1, R16.1, R18.1, R20.1, R28.2, R30.2, R31.2, R33.1, RV1.1, U2.2 (VO), U3.6 (VDD), U3.7 (VREGIN), U4.3 (3V3), U6.8 (VCCB); no longer SW1.2
- net at R29.1: now also U6.2 (A1); no longer J4.2 (Pin_2)
- net LED_OUT: no longer names the net of R29.2
- net LED_OUT: now also J4.2 (Pin_2)
- removed net Switch_in: C14.1, R1.2, R5.2
- new net: R22.1, U5.4 (PORT)
- new net: R21.2, U5.5 (VBUS_DET)
- new net: D3.1 (K), Q6.2 (D)
- new net: D8.1 (A1), J1.A4 (VBUS), J1.A9 (VBUS), J1.B4 (VBUS), J1.B9 (VBUS), Q2.1 (D), Q9.1 (D)
- new net: R38.1, U6.3 (A2)
- new net: J7.2 (Pin_2), R38.2
- new net: Q3.2 (G), R4.1
- new net: C17.1, Q2.3 (S), Q3.3 (S)
- new net: D4.1 (K), Q7.2 (D)
- new net: D4.2 (A), R18.2
- new net: D9.1 (A1), J2.2 (Pin_2), Q1.1 (D)
- new net: Q1.2 (G), R1.1
- new net: D3.2 (A), R16.2
- new net: Q5.1 (G), R11.1
- new net: Q4.1 (G), R10.1
- new net: D1.2 (A), R13.2
- new net: R8.1, U3.26 (TXD)
- new net: R7.2, U3.4 (D+)
- new net: R9.1, U3.25 (RXD)
- new net: R6.2, U3.5 (D-)
- new net: R26.2, R27.1, U3.8 (VBUS)
- new net: R5.2, U3.9 (~{RST})
- new net: Q9.2 (G), R25.1
- new net: D2.2 (A), R14.2
- new net: C24.1, J6.R, R32.1
- new net: C23.1, J6.T, R34.1
- new net: D5.2 (A), R20.2
- new net: D5.1 (K), Q8.2 (D)
- new net +1.65V: C22.1, R33.2, R35.1, R36.2, R37.2
- new net CC1: J1.A5 (CC1), U5.1 (CC1)
- new net EN/CHIP_PU: C5.1, Q4.2 (D), R12.1, TP1.1, U4.8 (EN/CHIP_PU)
- new net GPIO10: C14.1, J5.1 (Pin_1), R30.1, SW1.2, U4.16 (GPIO10)
- new net GPIO18: J3.8 (Pin_8), U4.26 (GPIO18/USB_D-)
- new net GPIO19: J3.5 (Pin_5), U4.27 (GPIO19/USB_D+)
- new net GPIO4/ADC1_CH4: C16.1, RV1.2, U4.18 (GPIO4/ADC1_CH4)
- new net GPIO5/ADC2_CH0: J3.2 (Pin_2), U4.19 (GPIO5/ADC2_CH0)
- new net GPIO6: Q8.1 (G), R19.1, U4.20 (GPIO6)
- new net GPIO7: R28.1, TP6.1, U4.21 (GPIO7), U5.6 (~{VCONN_FAULT})
- new net GPIO8: U4.22 (GPIO8), U6.6 (B2), U6.7 (B1)
- new net GPIO9/BOOT: Q5.2 (D), R31.1, TP7.1, U4.23 (GPIO9)
- new net LINE_INPUT_L: C23.2, D10.3 (K), R24.1, R37.1, U4.5 (GPIO2/ADC1_CH2)
- new net LINE_INPUT_R: C24.2, D11.3 (K), R23.1, R36.1, U4.6 (GPIO3/ADC1_CH3)
- new net U0RXD: Q7.1 (G), R17.1, R9.2, TP5.1, U4.30 (GPIO20/U0RXD)
- new net U0TXD: Q6.1 (G), R15.1, R8.2, TP4.1, U4.31 (GPIO21/U0TXD)
- new net USB_MODE_1: TP2.1, U4.12 (GPIO0/ADC1_CH0/XTAL_32K_P), U5.7 (OUT1)
- new net USB_MODE_2: TP3.1, U4.13 (GPIO1/ADC1_CH1/XTAL_32K_N), U5.8 (OUT2)
- new net VBUS: C8.1, Q9.3 (S), R21.1, R27.2, U5.12 (VDD)
- new net ~{DTR}: Q5.3 (S), R10.2, U3.28 (~{DTR})
- new net ~{RTS}: Q4.3 (S), R11.2, U3.24 (~{RTS})
- no-connect marks 0 -> 30
Other:
- note added: "ESP32 Flash auto program"
- note added: "ESP32 microcontroller module"
- note added: "GPIO headers"
- note added: "I_{LED} = 2.5mA V_{F} = 2.0-2.1V"
- note added: "Line audio input"
- note added: "Push button"
- note added: "SK6812RGBW output stage"
- note added: "Status LEDs"
- note added: "Trim potentiometer (firmware input)"
- note added: "USB to serial interface"
- note added: "USB-C 1.1 capabilities"
- note added: "USB-C receptacle Power path and regulation"
- title: ESP32-C3 based LED controller for WS2812/SK6812 -> ESP32-C3 based LED controller for SK6812
- moved on the sheet: C11, J1, J4, R29, SW1

Commit message: latest updates
Parts:
- C11, C19: footprint Capacitor_Tantalum_SMD:CP_EIA-3528-12_Kemet-T -> Capacitor_SMD:CP_Elec_8x6.7
- D8, D9: footprint Diode_SMD:D_SMA -> Diode_SMD:D_SMB
- J1: symbol Connector:USB_C_Receptacle -> Connector:USB_C_Receptacle_USB2.0_14P
- J2: value External supply -> +5V/GND in
- J3: footprint (none) -> Connector_PinHeader_2.54mm:PinHeader_1x09_P2.54mm_Vertical
- J4: value LED strip 1 -> SK6812RGBW
- J6: footprint Connector_Audio:Jack_3.5mm_PJ320D_Horizontal -> Connector_Audio:Jack_3.5mm_CUI_SJ-3523-SMT_Horizontal
- J7: value LED strip 2 -> SK6812RGBW; footprint Connector_PinHeader_2.54mm:PinHeader_1x03_P2.54mm_Horizontal -> TerminalBlock_RND:TerminalBlock_RND_205-00233_1x03_P5.08mm_Horizontal
- J8: value 5V 10A output -> +5V/GND out; footprint Connector_PinHeader_2.54mm:PinHeader_1x03_P2.54mm_Horizontal -> TerminalBlock_RND:TerminalBlock_RND_205-00232_1x02_P5.08mm_Horizontal
- Q9: footprint Package_TO_SOT_SMD:TO-252-2 -> Package_TO_SOT_SMD:SOT-23
- TP1, TP2, TP3, TP4, TP5, TP6, TP7: footprint (none) -> TestPoint:TestPoint_Pad_D3.0mm
Connections:
- net +5V: now also J7.3 (Pin_3), J8.2 (Pin_2); no longer J7.1 (Pin_1), J8.1 (Pin_1)
- net GND: now also J5.1 (Pin_1), J7.1 (Pin_1), J8.1 (Pin_1); no longer J5.2 (Pin_2), J7.3 (Pin_3), J8.2 (Pin_2)
- net GPIO10: now also J5.2 (Pin_2); no longer J5.1 (Pin_1)
- net VBUS_IN: now reaches D8.1 (A1), J1.A4 (VBUS), J1.A9 (VBUS), J1.B4 (VBUS), J1.B9 (VBUS), Q2.1 (D), Q9.1 (D)
- no-connect marks 30 -> 20
Other:
- moved on the sheet: J2, J7, J8
